File: pcb/5370.v3.1/5370.sch (KiCad schematic (older format))
At the start: 13 parts, among them P1 P1A, P2 P1B, U1 BEAGLEBONE_BLACK, U4 74LVC4245

Commit message: cleanup schematic
cleanup schematic in preparation for fabrication quotes
Parts:
- C2: renamed from C7; footprint ~ -> 5370-SM0805
- C3: renamed from C8; footprint ~ -> 5370-SM0805
- FB1: value 1KZ -> 30Z
- R1: footprint 5370-SM0805 -> 5370-BOURNS-4816P
- U1: footprint (none) -> 5370-BEAGLEBONE_BLACK
- renumbered R3 to R2, R4 to R3, U4 to U2
Other:
- note added: "Diode Vf = 240 mV\n@ If = 10 mA"
- note removed: "Vf = 240 mV"
- moved on the sheet: C1, C2, C3, D1, D2, FB1, P1, P2, R1, R2, R3, U1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
